Commit message: finalized lidar sim descreptions

File: transbot_description/urdf/lidar.xacro (robot description, xacro)
@@ -2,5 +2,5 @@
 <robot xmlns:xacro="http://www.ros.org/wiki/xacro">
     <joint name="laser_joint" type="fixed">
-        <origin xyz="0.0 0.0 0.0" rpy="0 0 0"/>
+        <origin xyz="0 0 0.135" rpy="0 0 0"/>
         <parent link="base_link"/>
         <child link="laser_frame"/>
@@ -8,5 +8,5 @@
     <link name="laser_frame">
         <visual>
-            <origin xyz="-0.0195 -0.035 0.088" rpy="1.570796327 0 3.14"/>
+            <origin xyz="-0.0195 -0.035 -0.047" rpy="1.570796327 0 3.14"/>
             <geometry>
                 <mesh filename="package://transbot_description/meshes/rplidar.STL" scale="0.001 0.001 0.001"/>
@@ -46,10 +46,10 @@
                 </scan>
                 <range>
-                    <min>0.3</min>
+                    <min>0.2</min>
                     <max>12.0</max>
                     <resolution>0.01</resolution>
                 </range>
             </ray>
-            <plugin name="gazebo_ros_laser" filename="libgazebo_ros_laser.so">
+            <plugin name="laser_controller" filename="libgazebo_ros_ray_sensor.so">
                 <ros>
                     <argument>~/out:=scan</argument>

File: transbot_description/urdf/mobile_base_gazebo.xacro (robot description, xacro)
@@ -4,4 +4,7 @@
     <gazebo reference="base_link">
         <material>Gazebo/Green</material>
+    </gazebo>
+    <gazebo reference="laser_frame">
+        <material>Gazebo/Grey</material>
     </gazebo>
     <gazebo reference="left_wheel_link">
